Commit message: Fix xacro mesh path

File: config/steward.urdf.xacro (robot description, xacro)
@@ -106,5 +106,5 @@
                 <origin xyz="0 0 0" rpy="0 0 ${side*PI/2}"/>
                 <geometry>
-                    <mesh filename="file:///home/main/Arbor/steward/data/meshes/steward/rocker.stl" />
+                    <mesh filename="file://$(arg mesh_path)/rocker.stl" />
                 </geometry>
                 <material name="${warthog_color}">
@@ -115,5 +115,5 @@
                 <origin xyz="0 0 0" rpy="0 0 ${side*PI/2}"/>
                 <geometry>
-                    <mesh filename="file:///home/main/Arbor/steward/data/meshes/steward/fenders.stl" />
+                    <mesh filename="file://$(arg mesh_path)/fenders.stl" />
                 </geometry>
                 <material name="${warthog_color}">
@@ -124,5 +124,5 @@
                 <origin xyz="0 0 0" rpy="0 0 ${side*PI/2}"/>
                 <geometry>
-                    <mesh filename="file:///home/main/Arbor/steward/data/meshes/steward/fenders.stl" />
+                    <mesh filename="file://$(arg mesh_path)/fenders.stl" />
                 </geometry>
             </collision>
@@ -140,5 +140,5 @@
                 <origin xyz="0 ${side*-0.0244} 0" rpy="0 0 0"/>
                 <geometry>
-                    <mesh filename="file:///home/main/Arbor/steward/data/meshes/steward/light.stl" />
+                    <mesh filename="file://$(arg mesh_path)/light.stl" />
                 </geometry>
                 <material name="white">
@@ -166,5 +166,5 @@
                 <origin xyz="0 ${side*-0.0244} 0" rpy="0 0 ${side*PI}"/>
                 <geometry>
-                    <mesh filename="file:///home/main/Arbor/steward/data/meshes/steward/light.stl" />
+                    <mesh filename="file://$(arg mesh_path)/light.stl" />
                 </geometry>
                 <material name="red">
@@ -212,5 +212,5 @@
                 <origin xyz="0 0 0" rpy="0 0 ${PI/2}"/>
                 <geometry>
-                    <mesh filename="file:///home/main/Arbor/steward/data/meshes/steward/wheel.stl" />
+                    <mesh filename="file://$(arg mesh_path)/wheel.stl" />
                 </geometry>
                 <material name="dark_grey" />

Commit message: Yeet

File: config/steward.urdf.xacro (robot description, xacro)
@@ -2,5 +2,5 @@
 <robot name="steward"
     xmlns:xacro="http://www.ros.org/wiki/xacro">
-    <xacro:property name="PI" value="3.1415926535897931"/>
+    <xacro:property name="PI" value="3.1415926535897931" />
     <xacro:property name="wheel_radius" value="0.3" />
     <xacro:property name="wheel_width" value="0.25" />
@@ -12,5 +12,5 @@
     <xacro:property name="diff_unit_length" value="1.34" />
     <xacro:property name="diff_unit_width" value="0.28" />
-    <xacro:property name="diff_unit_height" value="0.63"/>
+    <xacro:property name="diff_unit_height" value="0.63" />
     <xacro:property name="diff_unit_mass" value="50" />
     <xacro:property name="diff_unit_offset_x" value="0.00" />
@@ -21,5 +21,5 @@
     <xacro:property name="chassis_height" value="0.30" />
     <xacro:property name="chassis_mass" value="100" />
-    <xacro:property name="dummy_inertia" value="1e-09"/>
+    <xacro:property name="dummy_inertia" value="1e-09" />
     <xacro:property name="warthog_color" value="yellow" />
     <xacro:if value="${warthog_color == 'yellow'}">
@@ -36,8 +36,10 @@
     </xacro:if>
     <xacro:macro name="wheel_inertia" params="m r h">
-        <inertia ixx="${m*(3*r*r+h*h)/12}" ixy="0" ixz="0" iyy="${m*r*r/2}" iyz="0" izz="${m*(3*r*r+h*h)/12}" />
+        <inertia ixx="${m*(3*r*r+h*h)/12}" ixy="0" ixz="0" iyy="${m*r*r/2}" iyz="0"
+            izz="${m*(3*r*r+h*h)/12}" />
     </xacro:macro>
     <xacro:macro name="box_inertia" params="m x y z">
-        <inertia ixx="${m*(y*y+z*z)/12}" ixy="0" ixz="0" iyy="${m*(x*x+z*z)/12}" iyz="0" izz="${m*(x*x+z*z)/12}" />
+        <inertia ixx="${m*(y*y+z*z)/12}" ixy="0" ixz="0" iyy="${m*(x*x+z*z)/12}" iyz="0"
+            izz="${m*(x*x+z*z)/12}" />
     </xacro:macro>
     <material name="dark_grey">
@@ -62,10 +64,11 @@
     <link name="chassis_link">
         <inertial>
-            <origin xyz="0 0 0" rpy="0 0 0"/>
-            <mass value="${chassis_mass}"/>
-            <xacro:box_inertia m="${chassis_mass}" x="${chassis_length}" y="${chassis_width}" z="${chassis_height}" />
+            <origin xyz="0 0 0" rpy="0 0 0" />
+            <mass value="${chassis_mass}" />
+            <xacro:box_inertia m="${chassis_mass}" x="${chassis_length}" y="${chassis_width}"
+                z="${chassis_height}" />
         </inertial>
         <visual>
-            <origin xyz="0 0 0" rpy="0 0 0"/>
+            <origin xyz="0 0 0" rpy="0 0 0" />
             <geometry>
                 <mesh filename="file://$(arg mesh_path)/chassis.stl" />
@@ -76,5 +79,5 @@
         </visual>
         <visual>
-            <origin xyz="0 0 0" rpy="0 0 0"/>
+            <origin xyz="0 0 0" rpy="0 0 0" />
             <geometry>
                 <mesh filename="file://$(arg mesh_path)/e-stop.stl" />
@@ -85,5 +88,5 @@
         </visual>
         <collision>
-            <origin xyz="0 0 0" rpy="0 0 0"/>
+            <origin xyz="0 0 0" rpy="0 0 0" />
             <geometry>
                 <mesh filename="file://$(arg mesh_path)/chassis-collision.stl" />
@@ -93,16 +96,23 @@
     <joint name="base_link_joint" type="fixed">
         <origin xyz="0 0 0.025" rpy="0 0 0" />
-        <parent link="base_link"/>
+        <parent link="base_link" />
         <child link="chassis_link" />
+    </joint>
+    <link name="swiftnav-gnss"></link>
+    <joint name="gnss_joint" type="fixed">
+        <origin xyz="-0.25 -0.3 0.3" rpy="0 0 0" />
+        <parent link="base_link" />
+        <child link="swiftnav-gnss" />
     </joint>
     <xacro:macro name="diff_unit" params="prefix side left">
         <link name="${prefix}_diff_unit_link">
             <inertial>
-                <origin xyz="0 ${side*-1*0.05} 0.197" rpy="0 0 0"/>
-                <mass value="${diff_unit_mass}"/>
-                <xacro:box_inertia m="${diff_unit_mass}" x="${diff_unit_length}" y="${diff_unit_width}" z="${diff_unit_height}" />
+                <origin xyz="0 ${side*-1*0.05} 0.197" rpy="0 0 0" />
+                <mass value="${diff_unit_mass}" />
+                <xacro:box_inertia m="${diff_unit_mass}" x="${diff_unit_length}"
+                    y="${diff_unit_width}" z="${diff_unit_height}" />
             </inertial>
             <visual>
-                <origin xyz="0 0 0" rpy="0 0 ${side*PI/2}"/>
+                <origin xyz="0 0 0" rpy="0 0 ${side*PI/2}" />
                 <geometry>
                     <mesh filename="file://$(arg mesh_path)/rocker.stl" />
@@ -113,5 +123,5 @@
             </visual>
             <visual>
-                <origin xyz="0 0 0" rpy="0 0 ${side*PI/2}"/>
+                <origin xyz="0 0 0" rpy="0 0 ${side*PI/2}" />
                 <geometry>
                     <mesh filename="file://$(arg mesh_path)/fenders.stl" />
@@ -122,5 +132,5 @@
             </visual>
             <collision>
-                <origin xyz="0 0 0" rpy="0 0 ${side*PI/2}"/>
+                <origin xyz="0 0 0" rpy="0 0 ${side*PI/2}" />
                 <geometry>
                     <mesh filename="file://$(arg mesh_path)/fenders.stl" />
@@ -129,14 +139,15 @@
         </link>
         <joint name="${prefix}_diff_unit_joint" type="revolute">
-            <limit upper="0.4" lower="-0.4" effort="100" velocity="1"/>
-            <parent link="chassis_link"/>
-            <child link="${prefix}_diff_unit_link"/>
-            <origin xyz="${diff_unit_offset_x} ${diff_unit_offset_y*side} ${diff_unit_offset_z}" rpy="0 0 0" />
-            <axis xyz="0 1 0"/>
-            <dynamics damping="100" friction="0.5"/>
+            <limit upper="0.4" lower="-0.4" effort="100" velocity="1" />
+            <parent link="chassis_link" />
+            <child link="${prefix}_diff_unit_link" />
+            <origin xyz="${diff_unit_offset_x} ${diff_unit_offset_y*side} ${diff_unit_offset_z}"
+                rpy="0 0 0" />
+            <axis xyz="0 1 0" />
+            <dynamics damping="100" friction="0.5" />
         </joint>
         <link name="${prefix}_diff_unit_headlight_link">
             <visual>
-                <origin xyz="0 ${side*-0.0244} 0" rpy="0 0 0"/>
+                <origin xyz="0 ${side*-0.0244} 0" rpy="0 0 0" />
                 <geometry>
                     <mesh filename="file://$(arg mesh_path)/light.stl" />
@@ -150,5 +161,5 @@
             <parent link="${prefix}_diff_unit_link" />
             <child link="${prefix}_diff_unit_headlight_link" />
-            <origin xyz="0 0 0" rpy="0 0 0"/>
+            <origin xyz="0 0 0" rpy="0 0 0" />
         </joint>
         <gazebo reference="${prefix}_diff_unit_headlight_link">
@@ -164,5 +175,5 @@
         <link name="${prefix}_diff_unit_taillight_link">
             <visual>
-                <origin xyz="0 ${side*-0.0244} 0" rpy="0 0 ${side*PI}"/>
+                <origin xyz="0 ${side*-0.0244} 0" rpy="0 0 ${side*PI}" />
                 <geometry>
                     <mesh filename="file://$(arg mesh_path)/light.stl" />
@@ -176,5 +187,5 @@
             <parent link="${prefix}_diff_unit_link" />
             <child link="${prefix}_diff_unit_taillight_link" />
-            <origin xyz="0 0 0" rpy="0 0 0"/>
+            <origin xyz="0 0 0" rpy="0 0 0" />
         </joint>
         <gazebo reference="${prefix}_diff_unit_taillight_link">
@@ -200,6 +211,6 @@
         </gazebo>
     </xacro:macro>
-    <xacro:diff_unit prefix="left" side="1" left="true"/>
-    <xacro:diff_unit prefix="right" side="-1" left="false"/>
+    <xacro:diff_unit prefix="left" side="1" left="true" />
+    <xacro:diff_unit prefix="right" side="-1" left="false" />
     <xacro:macro name="wheel" params="prefix side *joint_pose">
         <link name="${prefix}_${side}_wheel_link">
@@ -210,5 +221,5 @@
             </inertial>
             <visual>
-                <origin xyz="0 0 0" rpy="0 0 ${PI/2}"/>
+                <origin xyz="0 0 0" rpy="0 0 ${PI/2}" />
                 <geometry>
                     <mesh filename="file://$(arg mesh_path)/wheel.stl" />
@@ -217,15 +228,15 @@
             </visual>
             <collision>
-                <origin xyz="0 0 0" rpy="${PI/2} 0 0"/>
-                <geometry>
-                    <cylinder radius="${wheel_radius}" length="${wheel_width}"/>
+                <origin xyz="0 0 0" rpy="${PI/2} 0 0" />
+                <geometry>
+                    <cylinder radius="${wheel_radius}" length="${wheel_width}" />
                 </geometry>
             </collision>
         </link>
         <joint name="${prefix}_${side}_wheel_joint" type="continuous">
-            <parent link="${side}_diff_unit_link"/>
-            <child link="${prefix}_${side}_wheel_link"/>
+            <parent link="${side}_diff_unit_link" />
+            <child link="${prefix}_${side}_wheel_link" />
             <xacro:insert_block name="joint_pose" />
-            <axis xyz="0 1 0"/>
+            <axis xyz="0 1 0" />
         </joint>
         <gazebo reference="${prefix}_${side}_wheel_link">

Commit message: Add GNSS transform pub

File: config/steward.urdf.xacro (robot description, xacro)
@@ -96,4 +96,10 @@
         <child link="chassis_link" />
     </joint>
+    <link name="swiftnav-gnss"></link>
+    <joint name="gnss_link_joint" type="fixed">
+        <origin xyz="-0.2 -0.3 0.5" rpy="0 0 0" />
+        <parent link="base_link"/>
+        <child link="swiftnav-gnss" />
+    </joint>
     <xacro:macro name="diff_unit" params="prefix side left">
         <link name="${prefix}_diff_unit_link">
